Commit message: update model

File: src/diff_drive_description/urdf/diff_drive.urdf.xacro (robot description, xacro)
@@ -26,4 +26,11 @@
             </collision>
         </link>
+        <gazebo reference = "${name}">
+            <visual>
+                <material>
+                    <ambient>${rgba}</ambient>
+                </material>
+            </visual>
+        </gazebo>
     </xacro:macro>
     <xacro:macro name = "make_cylinder_link"
@@ -53,8 +60,55 @@
             </collision>
         </link>
+        <gazebo reference = "${name}">
+            <visual>
+                <material>
+                    <ambient>${rgba}</ambient>
+                </material>
+            </visual>
+            <mu1 value = "1"/>
+            <mu2 value = "1"/>
+            <kp value="1000000"/>
+            <kd value= "100"/>
+        </gazebo>
+    </xacro:macro>
+    <xacro:macro name = "make_sphere_link"
+                 params = "name xyz rpy mass radius rgba">
+        <link name = "${name}">
+            <inertial>
+                <origin xyz = "${xyz}" rpy = "${rpy}"/>
+                <mass value="${mass}"/>
+                <inertia ixx="${(2/5) * mass * radius * radius}" ixy="0.0" ixz="0.0"
+                         iyy="${(2/5) * mass * radius * radius}" iyz="0.0"
+                         izz="${(2/5) * mass * radius * radius}"/>
+            </inertial>
+            <visual>
+                <origin xyz = "${xyz}" rpy = "${rpy}"/>
+                <geometry>
+                    <sphere radius="${radius}"/>
+                </geometry>
+                <material name = "${name}_material">
+                    <color rgba = "${rgba}"/>
+                </material>
+            </visual>
+            <collision>
+                <origin xyz = "${xyz}" rpy = "${rpy}"/>
+                <geometry>
+                    <sphere radius="${radius}"/>
+                </geometry>
+            </collision>
+        </link>
+        <gazebo reference = "${name}">
+            <visual>
+                <material>
+                    <ambient>${rgba}</ambient>
+                </material>
+            </visual>
+            <mu1 value="0" />
+            <mu2 value="0" />
+        </gazebo>
     </xacro:macro>
     <xacro:macro name = "make_continuous_joint"
-                 params = "name xyz rpy parent child axis damping friction">
-        <joint name = "${name}" type = "continuous">
+                 params = "name joint_type xyz rpy parent child axis damping friction">
+        <joint name = "${name}" type = "${joint_type}">
             <origin xyz = "${xyz}" rpy = "${rpy}"/>
             <parent link="${parent}"/>
@@ -64,22 +118,32 @@
         </joint>
     </xacro:macro>
+    <xacro:macro name = "make_fixed_joint"
+                 params = "name joint_type xyz rpy parent child damping friction">
+        <joint name = "${name}" type = "${joint_type}">
+            <origin xyz = "${xyz}" rpy = "${rpy}"/>
+            <parent link="${parent}"/>
+            <child link="${child}"/>
+            <dynamics damping = "${damping}" friction = "${friction}"/>
+        </joint>
+    </xacro:macro>
     <xacro:make_base_link name ="base_link"
                           xyz = "0 0 0"
                           rpy = "0 0 0"
-                          mass = "0.5"
+                          mass = "1"
                           width = "0.6"
                           height = "0.1"
                           depth = "0.4"
-                          rgba = "0.2 0.2 0.2 1.0"/>
+                          rgba = "1.0 1.0 1.0 0.2"/>
     <xacro:make_cylinder_link name = "left_wheel"
                            xyz = "0 0 0"
                            rpy = "0 0 0"
-                           mass = "0.1"
+                           mass = "0.05"
                            radius = "0.1"
                            length = "0.04"
                            rgba = "1 0.2 0.2 1.0"/>
     <xacro:make_continuous_joint name = "left_wheel_joint"
+                                 joint_type = "continuous"
                                  xyz = "-0.1 0.22 0"
-                                 rpy = "0.0 -1.57 -1.57"
+                                 rpy = "0 ${-pi/2} ${-pi/2}"
                                  parent = "base_link"
                                  child = "left_wheel"
@@ -90,11 +154,12 @@
                            xyz = "0 0 0"
                            rpy = "0 0 0"
-                           mass = "0.1"
+                           mass = "0.05"
                            radius = "0.1"
                            length = "0.04"
                            rgba = "1 0.2 0.2 1.0"/>
     <xacro:make_continuous_joint name = "right_wheel_joint"
+                                 joint_type = "continuous"
                                  xyz = "-0.1 -0.22 0"
-                                 rpy = "0.0 -1.57 -1.57"
+                                 rpy = "0.0 ${-pi/2} ${-pi/2}"
                                  parent = "base_link"
                                  child = "right_wheel"
@@ -102,33 +167,48 @@
                                  damping = "0"
                                  friction = "0"/>
-    <xacro:make_cylinder_link name = "cluster_support"
-                                 xyz = "0 0 0"
-                                 rpy = "0 0 0"
-                                 mass = "0.1"
-                                 radius = "0.02"
-                                 length = "0.1"
-                                 rgba = "0.2 1.0 0.2 1.0"/>
-    <xacro:make_continuous_joint name = "cluster_support_joint"
-                                 xyz = "0.32 0 0"
-                                 rpy = "0 0 0"
-                                 parent = "base_link"
-                                 child = "cluster_support"
-                                 axis = "0 0 1"
-                                 damping = "0"
-                                 friction = "0"/>
-    <xacro:make_cylinder_link name = "cluster_wheel"
+    <xacro:make_sphere_link name = "cluster_wheel"
                                  xyz = "0 0 0"
                                  rpy = "0 0 0"
                                  mass = "0.02"
-                                 radius = "0.025"
-                                 length = "0.01"
+                                 radius = "0.05"
                                  rgba = "0.2 0.2 1.0 1.0"/>
-    <xacro:make_continuous_joint name = "cluster_wheel_joint"
-                                 xyz = "0 0 -0.075"
-                                 rpy = "0 -1.57 -1.57"
-                                 parent = "cluster_support"
+    <xacro:make_fixed_joint name = "cluster_wheel_joint"
+                                 joint_type = "fixed"
+                                 xyz = "0.26 0 -0.05"
+                                 rpy = "0 0 0"
+                                 parent = "base_link"
                                  child = "cluster_wheel"
-                                 axis = "0 0 1"
                                  damping = "0"
                                  friction = "0"/>
+    <xacro:macro name = "make_simple_transmission"
+                 params = "name
+                           joint
+                           hardware_interface
+                           actuator
+                           mechanical_reduction">
+        <transmission name = "${joint}">
+            <type>transmission_interface/SimpleTransmission</type>
+            <joint name = "${joint}">
+                <hardwareInterface>${hardware_interface}</hardwareInterface>
+            </joint>
+            <actuator name = "${actuator}">
+                <mechanicalReduction>${mechanical_reduction}</mechanicalReduction>
+            </actuator>
+        </transmission>
+    </xacro:macro>
+    <xacro:make_simple_transmission name = "left_wheel_transmission"
+                                    joint = "left_wheel_joint"
+                                    hardware_interface = "hardware_interface/VelocityJointInterface"
+                                    actuator = "left_motor"
+                                    mechanical_reduction = "1"/>
+    <xacro:make_simple_transmission name = "right_wheel_transmission"
+                                    joint = "right_wheel_joint"
+                                    hardware_interface = "hardware_interface/VelocityJointInterface"
+                                    actuator = "right_motor"
+                                    mechanical_reduction = "1"/>
+    <gazebo>
+        <plugin name="gazebo_ros_control" filename="libgazebo_ros_control.so">
+            <robotNamespace>/</robotNamespace>
+        </plugin>
+    </gazebo>
 </robot>

Commit message: update pid

File: src/diff_drive_description/urdf/diff_drive.urdf.xacro (robot description, xacro)
@@ -127,4 +127,10 @@
         </joint>
     </xacro:macro>
+    <link name="dummy">
+    </link>
+    <joint name="dummy_joint" type="fixed">
+        <parent link="dummy"/>
+        <child link="base_link"/>
+    </joint>
     <xacro:make_base_link name ="base_link"
                           xyz = "0 0 0"
